File: TrigInOutPu.sch (KiCad schematic (older format))
At the start: 7 parts, among them P7 BNC, P8 BNC, U3 ISO1540

Commit message: Fixed some annotations and footprints
Parts:
- P7, P8: footprint Connectors_TE-Connectivity:BNC_Socket_TYCO-AMP_LargePads -> lib_fp:BNC_Socket_RSpro_LargePads
- renumbered C5 to C1, C7 to C2, R12 to R10, R13 to R11, U3 to U2
Connections:
- net +3V3: now also R10.2, R11.2
