File: TrigInOutPu.sch (KiCad schematic (older format))
At the start: 7 parts, among them P7 BNC, P8 BNC, U2 ISO1540

Commit message: Cleanups
Parts:
- U2: footprint Housings_SOIC:SOIC-8-1EP_3.9x4.9mm_Pitch1.27mm -> Housings_SOIC:SOIC-8_3.9x4.9mm_Pitch1.27mm
Changed lines of the file:
@@
 AR Path="/59B431E3/59A9A587" Ref="P9"  Part="1"
 AR Path="/59B46FD6/59A9A587" Ref="P11"  Part="1"
-F 0 "P7" H 1710 1020 50  0000 C CNN
+F 0 "P11" H 1710 1020 50  0000 C CNN
 F 1 "BNC" V 1810 840 50  0000 C CNN
 F 2 "lib_fp:BNC_Socket_RSpro_LargePads" H 1700 900 50  0001 C CNN
@@
 AR Path="/59B431E3/59A9A58E" Ref="#PWR057"  Part="1"
 AR Path="/59B46FD6/59A9A58E" Ref="#PWR081"  Part="1"
-F 0 "#PWR033" H 1700 850 50  0001 C CNN
+F 0 "#PWR081" H 1700 850 50  0001 C CNN
 F 1 "GND" H 1700 950 50  0000 C CNN
 F 2 "" H 1700 1100 50  0000 C CNN
@@
 AR Path="/59B431E3/59B40E58" Ref="U5"  Part="1"
 AR Path="/59B46FD6/59B40E58" Ref="U8"  Part="1"
-F 0 "U2" H 5500 1200 60  0000 C CNN
+F 0 "U8" H 5500 1200 60  0000 C CNN
 F 1 "ISO1540" H 5500 800 60  0000 C CNN
-F 2 "Housings_SOIC:SOIC-8-1EP_3.9x4.9mm_Pitch1.27mm" H 5500 1000 60  0001 C CNN
+F 2 "Housings_SOIC:SOIC-8_3.9x4.9mm_Pitch1.27mm" H 5500 1000 60  0001 C CNN
 F 3 "" H 5500 1000 60  0001 C CNN
 	1    5500 1000
@@
 AR Path="/59B431E3/59B41346" Ref="#PWR058"  Part="1"
 AR Path="/59B46FD6/59B41346" Ref="#PWR082"  Part="1"
-F 0 "#PWR034" H 6100 750 50  0001 C CNN
+F 0 "#PWR082" H 6100 750 50  0001 C CNN
 F 1 "+5V" H 6100 1040 50  0000 C CNN
 F 2 "" H 6100 900 50  0001 C CNN
@@
 AR Path="/59B431E3/59B4138C" Ref="#PWR059"  Part="1"
 AR Path="/59B46FD6/59B4138C" Ref="#PWR083"  Part="1"
-F 0 "#PWR035" H 6100 850 50  0001 C CNN
+F 0 "#PWR083" H 6100 850 50  0001 C CNN
 F 1 "GND" H 6100 950 50  0000 C CNN
 F 2 "" H 6100 1100 50  0001 C CNN
@@
 AR Path="/59B431E3/59B4140C" Ref="#PWR060"  Part="1"
 AR Path="/59B46FD6/59B4140C" Ref="#PWR084"  Part="1"
-F 0 "#PWR036" H 4900 850 50  0001 C CNN
+F 0 "#PWR084" H 4900 850 50  0001 C CNN
 F 1 "GND" H 4900 950 50  0000 C CNN
 F 2 "" H 4900 1100 50  0001 C CNN
@@
 AR Path="/59B431E3/59B41431" Ref="#PWR061"  Part="1"
 AR Path="/59B46FD6/59B41431" Ref="#PWR085"  Part="1"
-F 0 "#PWR037" H 4900 750 50  0001 C CNN
+F 0 "#PWR085" H 4900 750 50  0001 C CNN
 F 1 "+3.3V" H 4900 1040 50  0000 C CNN
 F 2 "" H 4900 900 50  0001 C CNN
@@
 AR Path="/59B431E3/59B4156A" Ref="R18"  Part="1"
 AR Path="/59B46FD6/59B4156A" Ref="R26"  Part="1"
-F 0 "R10" V 4780 1250 50  0000 C CNN
+F 0 "R26" V 4780 1250 50  0000 C CNN
 F 1 "2k" V 4700 1250 50  0000 C CNN
 F 2 "Resistors_SMD:R_0603_HandSoldering" V 4630 1250 50  0001 C CNN
@@
 AR Path="/59B431E3/59B419CB" Ref="P10"  Part="1"
 AR Path="/59B46FD6/59B419CB" Ref="P12"  Part="1"
-F 0 "P8" H 1710 2170 50  0000 C CNN
+F 0 "P12" H 1710 2170 50  0000 C CNN
 F 1 "BNC" V 1810 1990 50  0000 C CNN
 F 2 "lib_fp:BNC_Socket_RSpro_LargePads" H 1700 2050 50  0001 C CNN
@@
 AR Path="/59B431E3/59B419D1" Ref="#PWR062"  Part="1"
 AR Path="/59B46FD6/59B419D1" Ref="#PWR086"  Part="1"
-F 0 "#PWR038" H 1700 2000 50  0001 C CNN
+F 0 "#PWR086" H 1700 2000 50  0001 C CNN
 F 1 "GND" H 1700 2100 50  0000 C CNN
 F 2 "" H 1700 2250 50  0000 C CNN
@@
 AR Path="/59B431E3/59B419E7" Ref="#PWR063"  Part="1"
 AR Path="/59B46FD6/59B419E7" Ref="#PWR087"  Part="1"
-F 0 "#PWR039" H 6100 1900 50  0001 C CNN
+F 0 "#PWR087" H 6100 1900 50  0001 C CNN
 F 1 "+5V" H 6100 2190 50  0000 C CNN
 F 2 "" H 6100 2050 50  0001 C CNN
@@
 AR Path="/59B431E3/59B419EE" Ref="#PWR064"  Part="1"
 AR Path="/59B46FD6/59B419EE" Ref="#PWR088"  Part="1"
-F 0 "#PWR040" H 6100 2000 50  0001 C CNN
+F 0 "#PWR088" H 6100 2000 50  0001 C CNN
 F 1 "GND" H 6100 2100 50  0000 C CNN
 F 2 "" H 6100 2250 50  0001 C CNN
@@
 AR Path="/59B431E3/59B419F4" Ref="#PWR065"  Part="1"
 AR Path="/59B46FD6/59B419F4" Ref="#PWR089"  Part="1"
-F 0 "#PWR041" H 4900 2000 50  0001 C CNN
+F 0 "#PWR089" H 4900 2000 50  0001 C CNN
 F 1 "GND" H 4900 2100 50  0000 C CNN
 F 2 "" H 4900 2250 50  0001 C CNN
@@
 AR Path="/59B431E3/59B419FA" Ref="#PWR066"  Part="1"
 AR Path="/59B46FD6/59B419FA" Ref="#PWR090"  Part="1"
-F 0 "#PWR042" H 4900 1900 50  0001 C CNN
+F 0 "#PWR090" H 4900 1900 50  0001 C CNN
 F 1 "+3.3V" H 4900 2190 50  0000 C CNN
 F 2 "" H 4900 2050 50  0001 C CNN
@@
 AR Path="/59B431E3/59B41A04" Ref="R19"  Part="1"
 AR Path="/59B46FD6/59B41A04" Ref="R27"  Part="1"
-F 0 "R11" V 4780 2400 50  0000 C CNN
+F 0 "R27" V 4780 2400 50  0000 C CNN
 F 1 "2k" V 4700 2400 50  0000 C CNN
 F 2 "Resistors_SMD:R_0603_HandSoldering" V 4630 2400 50  0001 C CNN
@@
 AR Path="/59B431E3/59B41AB2" Ref="U5"  Part="2"
 AR Path="/59B46FD6/59B41AB2" Ref="U8"  Part="2"
-F 0 "U2" H 5500 2350 60  0000 C CNN
+F 0 "U8" H 5500 2350 60  0000 C CNN
 F 1 "ISO1540" H 5500 1950 60  0000 C CNN
-F 2 "Housings_SOIC:SOIC-8-1EP_3.9x4.9mm_Pitch1.27mm" H 5500 2150 60  0001 C CNN
+F 2 "Housings_SOIC:SOIC-8_3.9x4.9mm_Pitch1.27mm" H 5500 2150 60  0001 C CNN
 F 3 "" H 5500 2150 60  0001 C CNN
 	2    5500 2150
@@
 AR Path="/59B431E3/59B41E6C" Ref="C4"  Part="1"
 AR Path="/59B46FD6/59B41E6C" Ref="C6"  Part="1"
-F 0 "C2" H 7425 1100 50  0000 L CNN
+F 0 "C6" H 7425 1100 50  0000 L CNN
 F 1 "100n" H 7425 900 50  0000 L CNN
 F 2 "Capacitors_SMD:C_0603_HandSoldering" H 7438 850 50  0001 C CNN
@@
 AR Path="/59B431E3/59B41E72" Ref="C3"  Part="1"
 AR Path="/59B46FD6/59B41E72" Ref="C5"  Part="1"
-F 0 "C1" H 7125 1100 50  0000 L CNN
+F 0 "C5" H 7125 1100 50  0000 L CNN
 F 1 "100n" H 7125 900 50  0000 L CNN
 F 2 "Capacitors_SMD:C_0603_HandSoldering" H 7138 850 50  0001 C CNN
@@
 AR Path="/59B431E3/59B41E78" Ref="#PWR067"  Part="1"
 AR Path="/59B46FD6/59B41E78" Ref="#PWR091"  Part="1"
-F 0 "#PWR043" H 7100 1000 50  0001 C CNN
+F 0 "#PWR091" H 7100 1000 50  0001 C CNN
 F 1 "GND" H 7100 1100 50  0000 C CNN
 F 2 "" H 7100 1250 50  0001 C CNN
@@
 AR Path="/59B431E3/59B41E7E" Ref="#PWR068"  Part="1"
 AR Path="/59B46FD6/59B41E7E" Ref="#PWR092"  Part="1"
-F 0 "#PWR044" H 7400 600 50  0001 C CNN
+F 0 "#PWR092" H 7400 600 50  0001 C CNN
 F 1 "+5V" H 7400 890 50  0000 C CNN
 F 2 "" H 7400 750 50  0001 C CNN
@@
 AR Path="/59B431E3/59B41E84" Ref="#PWR069"  Part="1"
 AR Path="/59B46FD6/59B41E84" Ref="#PWR093"  Part="1"
-F 0 "#PWR045" H 7100 600 50  0001 C CNN
+F 0 "#PWR093" H 7100 600 50  0001 C CNN
 F 1 "+3.3V" H 7100 890 50  0000 C CNN
 F 2 "" H 7100 750 50  0001 C CNN
@@
 AR Path="/59B431E3/59B41E8A" Ref="#PWR070"  Part="1"
 AR Path="/59B46FD6/59B41E8A" Ref="#PWR094"  Part="1"
-F 0 "#PWR046" H 7400 1000 50  0001 C CNN
+F 0 "#PWR094" H 7400 1000 50  0001 C CNN
 F 1 "GND" H 7400 1100 50  0000 C CNN
 F 2 "" H 7400 1250 50  0001 C CNN
@@
 AR Path="/59B431E3/59B91282" Ref="#PWR071"  Part="1"
 AR Path="/59B46FD6/59B91282" Ref="#PWR095"  Part="1"
-F 0 "#PWR047" H 4700 1350 50  0001 C CNN
+F 0 "#PWR095" H 4700 1350 50  0001 C CNN
 F 1 "+3.3V" H 4700 1640 50  0000 C CNN
 F 2 "" H 4700 1500 50  0001 C CNN
@@
 AR Path="/59B431E3/59B912BD" Ref="#PWR072"  Part="1"
 AR Path="/59B46FD6/59B912BD" Ref="#PWR096"  Part="1"
-F 0 "#PWR048" H 4700 2500 50  0001 C CNN
+F 0 "#PWR096" H 4700 2500 50  0001 C CNN
 F 1 "+3.3V" H 4700 2790 50  0000 C CNN
 F 2 "" H 4700 2650 50  0001 C CNN

Commit message: Cleanup teensy schematic and remove old custom.lib
Changed lines of the file:
@@
 EESchema Schematic File Version 2
+LIBS:teensy36_no-center
+LIBS:ldd-1000h
 LIBS:maxim
 LIBS:dmc2700
 LIBS:iso1540
 LIBS:74lvc
-LIBS:custom
 LIBS:ledflashcontroller-rescue
 LIBS:power
@@
 AR Path="/59B431E3/59A9A587" Ref="P9"  Part="1"
 AR Path="/59B46FD6/59A9A587" Ref="P11"  Part="1"
-F 0 "P11" H 1710 1020 50  0000 C CNN
+F 0 "P7" H 1710 1020 50  0000 C CNN
 F 1 "BNC" V 1810 840 50  0000 C CNN
 F 2 "lib_fp:BNC_Socket_RSpro_LargePads" H 1700 900 50  0001 C CNN
@@
 AR Path="/59B431E3/59A9A58E" Ref="#PWR057"  Part="1"
 AR Path="/59B46FD6/59A9A58E" Ref="#PWR081"  Part="1"
-F 0 "#PWR081" H 1700 850 50  0001 C CNN
+F 0 "#PWR033" H 1700 850 50  0001 C CNN
 F 1 "GND" H 1700 950 50  0000 C CNN
 F 2 "" H 1700 1100 50  0000 C CNN
@@
 AR Path="/59B431E3/59B40E58" Ref="U5"  Part="1"
 AR Path="/59B46FD6/59B40E58" Ref="U8"  Part="1"
-F 0 "U8" H 5500 1200 60  0000 C CNN
+F 0 "U2" H 5500 1200 60  0000 C CNN
 F 1 "ISO1540" H 5500 800 60  0000 C CNN
 F 2 "Housings_SOIC:SOIC-8_3.9x4.9mm_Pitch1.27mm" H 5500 1000 60  0001 C CNN
@@
 AR Path="/59B431E3/59B41346" Ref="#PWR058"  Part="1"
 AR Path="/59B46FD6/59B41346" Ref="#PWR082"  Part="1"
-F 0 "#PWR082" H 6100 750 50  0001 C CNN
+F 0 "#PWR034" H 6100 750 50  0001 C CNN
 F 1 "+5V" H 6100 1040 50  0000 C CNN
 F 2 "" H 6100 900 50  0001 C CNN
@@
 AR Path="/59B431E3/59B4138C" Ref="#PWR059"  Part="1"
 AR Path="/59B46FD6/59B4138C" Ref="#PWR083"  Part="1"
-F 0 "#PWR083" H 6100 850 50  0001 C CNN
+F 0 "#PWR035" H 6100 850 50  0001 C CNN
 F 1 "GND" H 6100 950 50  0000 C CNN
 F 2 "" H 6100 1100 50  0001 C CNN
@@
 AR Path="/59B431E3/59B4140C" Ref="#PWR060"  Part="1"
 AR Path="/59B46FD6/59B4140C" Ref="#PWR084"  Part="1"
-F 0 "#PWR084" H 4900 850 50  0001 C CNN
+F 0 "#PWR036" H 4900 850 50  0001 C CNN
 F 1 "GND" H 4900 950 50  0000 C CNN
 F 2 "" H 4900 1100 50  0001 C CNN
@@
 AR Path="/59B431E3/59B41431" Ref="#PWR061"  Part="1"
 AR Path="/59B46FD6/59B41431" Ref="#PWR085"  Part="1"
-F 0 "#PWR085" H 4900 750 50  0001 C CNN
+F 0 "#PWR037" H 4900 750 50  0001 C CNN
 F 1 "+3.3V" H 4900 1040 50  0000 C CNN
 F 2 "" H 4900 900 50  0001 C CNN
@@
 AR Path="/59B431E3/59B4156A" Ref="R18"  Part="1"
 AR Path="/59B46FD6/59B4156A" Ref="R26"  Part="1"
-F 0 "R26" V 4780 1250 50  0000 C CNN
+F 0 "R10" V 4780 1250 50  0000 C CNN
 F 1 "2k" V 4700 1250 50  0000 C CNN
 F 2 "Resistors_SMD:R_0603_HandSoldering" V 4630 1250 50  0001 C CNN
@@
 AR Path="/59B431E3/59B419CB" Ref="P10"  Part="1"
 AR Path="/59B46FD6/59B419CB" Ref="P12"  Part="1"
-F 0 "P12" H 1710 2170 50  0000 C CNN
+F 0 "P8" H 1710 2170 50  0000 C CNN
 F 1 "BNC" V 1810 1990 50  0000 C CNN
 F 2 "lib_fp:BNC_Socket_RSpro_LargePads" H 1700 2050 50  0001 C CNN
@@
 AR Path="/59B431E3/59B419D1" Ref="#PWR062"  Part="1"
 AR Path="/59B46FD6/59B419D1" Ref="#PWR086"  Part="1"
-F 0 "#PWR086" H 1700 2000 50  0001 C CNN
+F 0 "#PWR038" H 1700 2000 50  0001 C CNN
 F 1 "GND" H 1700 2100 50  0000 C CNN
 F 2 "" H 1700 2250 50  0000 C CNN
@@
 AR Path="/59B431E3/59B419E7" Ref="#PWR063"  Part="1"
 AR Path="/59B46FD6/59B419E7" Ref="#PWR087"  Part="1"
-F 0 "#PWR087" H 6100 1900 50  0001 C CNN
+F 0 "#PWR039" H 6100 1900 50  0001 C CNN
 F 1 "+5V" H 6100 2190 50  0000 C CNN
 F 2 "" H 6100 2050 50  0001 C CNN
@@
 AR Path="/59B431E3/59B419EE" Ref="#PWR064"  Part="1"
 AR Path="/59B46FD6/59B419EE" Ref="#PWR088"  Part="1"
-F 0 "#PWR088" H 6100 2000 50  0001 C CNN
+F 0 "#PWR040" H 6100 2000 50  0001 C CNN
 F 1 "GND" H 6100 2100 50  0000 C CNN
 F 2 "" H 6100 2250 50  0001 C CNN
@@
 AR Path="/59B431E3/59B419F4" Ref="#PWR065"  Part="1"
 AR Path="/59B46FD6/59B419F4" Ref="#PWR089"  Part="1"
-F 0 "#PWR089" H 4900 2000 50  0001 C CNN
+F 0 "#PWR041" H 4900 2000 50  0001 C CNN
 F 1 "GND" H 4900 2100 50  0000 C CNN
 F 2 "" H 4900 2250 50  0001 C CNN
@@
 AR Path="/59B431E3/59B419FA" Ref="#PWR066"  Part="1"
 AR Path="/59B46FD6/59B419FA" Ref="#PWR090"  Part="1"
-F 0 "#PWR090" H 4900 1900 50  0001 C CNN
+F 0 "#PWR042" H 4900 1900 50  0001 C CNN
 F 1 "+3.3V" H 4900 2190 50  0000 C CNN
 F 2 "" H 4900 2050 50  0001 C CNN
@@
 AR Path="/59B431E3/59B41A04" Ref="R19"  Part="1"
 AR Path="/59B46FD6/59B41A04" Ref="R27"  Part="1"
-F 0 "R27" V 4780 2400 50  0000 C CNN
+F 0 "R11" V 4780 2400 50  0000 C CNN
 F 1 "2k" V 4700 2400 50  0000 C CNN
 F 2 "Resistors_SMD:R_0603_HandSoldering" V 4630 2400 50  0001 C CNN
@@
 AR Path="/59B431E3/59B41AB2" Ref="U5"  Part="2"
 AR Path="/59B46FD6/59B41AB2" Ref="U8"  Part="2"
-F 0 "U8" H 5500 2350 60  0000 C CNN
+F 0 "U2" H 5500 2350 60  0000 C CNN
 F 1 "ISO1540" H 5500 1950 60  0000 C CNN
 F 2 "Housings_SOIC:SOIC-8_3.9x4.9mm_Pitch1.27mm" H 5500 2150 60  0001 C CNN
@@
 AR Path="/59B431E3/59B41E6C" Ref="C4"  Part="1"
 AR Path="/59B46FD6/59B41E6C" Ref="C6"  Part="1"
-F 0 "C6" H 7425 1100 50  0000 L CNN
+F 0 "C2" H 7425 1100 50  0000 L CNN
 F 1 "100n" H 7425 900 50  0000 L CNN
 F 2 "Capacitors_SMD:C_0603_HandSoldering" H 7438 850 50  0001 C CNN
@@
 AR Path="/59B431E3/59B41E72" Ref="C3"  Part="1"
 AR Path="/59B46FD6/59B41E72" Ref="C5"  Part="1"
-F 0 "C5" H 7125 1100 50  0000 L CNN
+F 0 "C1" H 7125 1100 50  0000 L CNN
 F 1 "100n" H 7125 900 50  0000 L CNN
 F 2 "Capacitors_SMD:C_0603_HandSoldering" H 7138 850 50  0001 C CNN
@@
 AR Path="/59B431E3/59B41E78" Ref="#PWR067"  Part="1"
 AR Path="/59B46FD6/59B41E78" Ref="#PWR091"  Part="1"
-F 0 "#PWR091" H 7100 1000 50  0001 C CNN
+F 0 "#PWR043" H 7100 1000 50  0001 C CNN
 F 1 "GND" H 7100 1100 50  0000 C CNN
 F 2 "" H 7100 1250 50  0001 C CNN
@@
 AR Path="/59B431E3/59B41E7E" Ref="#PWR068"  Part="1"
 AR Path="/59B46FD6/59B41E7E" Ref="#PWR092"  Part="1"
-F 0 "#PWR092" H 7400 600 50  0001 C CNN
+F 0 "#PWR044" H 7400 600 50  0001 C CNN
 F 1 "+5V" H 7400 890 50  0000 C CNN
 F 2 "" H 7400 750 50  0001 C CNN
@@
 AR Path="/59B431E3/59B41E84" Ref="#PWR069"  Part="1"
 AR Path="/59B46FD6/59B41E84" Ref="#PWR093"  Part="1"
-F 0 "#PWR093" H 7100 600 50  0001 C CNN
+F 0 "#PWR045" H 7100 600 50  0001 C CNN
 F 1 "+3.3V" H 7100 890 50  0000 C CNN
 F 2 "" H 7100 750 50  0001 C CNN
@@
 AR Path="/59B431E3/59B41E8A" Ref="#PWR070"  Part="1"
 AR Path="/59B46FD6/59B41E8A" Ref="#PWR094"  Part="1"
-F 0 "#PWR094" H 7400 1000 50  0001 C CNN
+F 0 "#PWR046" H 7400 1000 50  0001 C CNN
 F 1 "GND" H 7400 1100 50  0000 C CNN
 F 2 "" H 7400 1250 50  0001 C CNN
@@
 AR Path="/59B431E3/59B91282" Ref="#PWR071"  Part="1"
 AR Path="/59B46FD6/59B91282" Ref="#PWR095"  Part="1"
-F 0 "#PWR095" H 4700 1350 50  0001 C CNN
+F 0 "#PWR047" H 4700 1350 50  0001 C CNN
 F 1 "+3.3V" H 4700 1640 50  0000 C CNN
 F 2 "" H 4700 1500 50  0001 C CNN
@@
 AR Path="/59B431E3/59B912BD" Ref="#PWR072"  Part="1"
 AR Path="/59B46FD6/59B912BD" Ref="#PWR096"  Part="1"
-F 0 "#PWR096" H 4700 2500 50  0001 C CNN
+F 0 "#PWR048" H 4700 2500 50  0001 C CNN
 F 1 "+3.3V" H 4700 2790 50  0000 C CNN
 F 2 "" H 4700 2650 50  0001 C CNN
